Commit message: feat: Add remaining segments and joints for legs 2-5 in hexapod URDF

File: models/hexapod.urdf (robot description, URDF)
Before this commit: robot hexapod, 18 links, 17 joints
Links:
- added link leg2_segment2, mass 0.05; collision box size=0.1 0.2 0.1; visual box size=0.1 0.2 0.1
- added link leg2_segment3, mass 0.05; collision box size=0.1 0.2 0.1; visual box size=0.1 0.2 0.1
- added link leg3_segment2, mass 0.05; collision box size=0.1 0.2 0.1; visual box size=0.1 0.2 0.1
- added link leg3_segment3, mass 0.05; collision box size=0.1 0.2 0.1; visual box size=0.1 0.2 0.1
- added link leg4_segment1, mass 0.05; collision box size=0.1 0.2 0.1; visual box size=0.1 0.2 0.1
- added link leg4_segment2, mass 0.05; collision box size=0.1 0.2 0.1; visual box size=0.1 0.2 0.1
- added link leg4_segment3, mass 0.05; collision box size=0.1 0.2 0.1; visual box size=0.1 0.2 0.1
- added link leg5_segment1, mass 0.05; collision box size=0.1 0.2 0.1; visual box size=0.1 0.2 0.1
- added link leg5_segment2, mass 0.05; collision box size=0.1 0.2 0.1; visual box size=0.1 0.2 0.1
- added link leg5_segment3, mass 0.05; collision box size=0.1 0.2 0.1; visual box size=0.1 0.2 0.1
Joints:
- added joint leg2_joint2: type revolute, parent leg2_segment1, child leg2_segment2, origin xyz=0 0.12 0 rpy=0 0 0, axis 1 0 0, limit lower=0 upper=1.047 effort=10 velocity=1
- added joint leg2_joint3: type revolute, parent leg2_segment2, child leg2_segment3, origin xyz=0 0.12 0 rpy=0 0 0, axis 1 0 0, limit lower=0 upper=1.047 effort=10 velocity=1
- added joint leg3_joint2: type revolute, parent leg3_segment1, child leg3_segment2, origin xyz=0 0.12 0 rpy=0 0 0, axis 1 0 0, limit lower=0 upper=1.047 effort=10 velocity=1
- added joint leg3_joint3: type revolute, parent leg3_segment2, child leg3_segment3, origin xyz=0 0.12 0 rpy=0 0 0, axis 1 0 0, limit lower=0 upper=1.047 effort=10 velocity=1
- added joint leg4_joint1: type revolute, parent leg4_segment0, child leg4_segment1, origin xyz=0 0.12 0 rpy=0 0 0, axis 0 1 0, limit lower=-0.785 upper=0.785 effort=10 velocity=1
- added joint leg4_joint2: type revolute, parent leg4_segment1, child leg4_segment2, origin xyz=0 0.12 0 rpy=0 0 0, axis 1 0 0, limit lower=0 upper=1.047 effort=10 velocity=1
- added joint leg4_joint3: type revolute, parent leg4_segment2, child leg4_segment3, origin xyz=0 0.12 0 rpy=0 0 0, axis 1 0 0, limit lower=0 upper=1.047 effort=10 velocity=1
- added joint leg5_joint1: type revolute, parent leg5_segment0, child leg5_segment1, origin xyz=0 0.12 0 rpy=0 0 0, axis 0 1 0, limit lower=-0.785 upper=0.785 effort=10 velocity=1
- added joint leg5_joint2: type revolute, parent leg5_segment1, child leg5_segment2, origin xyz=0 0.12 0 rpy=0 0 0, axis 1 0 0, limit lower=0 upper=1.047 effort=10 velocity=1
- added joint leg5_joint3: type revolute, parent leg5_segment2, child leg5_segment3, origin xyz=0 0.12 0 rpy=0 0 0, axis 1 0 0, limit lower=0 upper=1.047 effort=10 velocity=1

Commit message: feat: Refactor hexapod URDF to standardize leg naming and improve material definitions

File: models/hexapod.urdf (robot description, URDF)
Before this commit: robot hexapod, 28 links, 27 joints
Links:
- removed link base_link
- removed link left_eye
- removed link leg0_segment0
- removed link leg0_segment1
- removed link leg0_segment2
- removed link leg0_segment3
- removed link leg1_segment0
- removed link leg1_segment1
- removed link leg1_segment2
- removed link leg1_segment3
- removed link leg2_segment0
- removed link leg2_segment1
- removed link leg2_segment2
- removed link leg2_segment3
- removed link leg3_segment0
- removed link leg3_segment1
- removed link leg3_segment2
- removed link leg3_segment3
- removed link leg4_segment0
- removed link leg4_segment1
- removed link leg4_segment2
- removed link leg4_segment3
- removed link leg5_segment0
- removed link leg5_segment1
- removed link leg5_segment2
- removed link leg5_segment3
- removed link right_eye
- added link body, mass 1.0; collision box size=1.0 0.4 0.2; visual box size=1.0 0.4 0.2
- added link eye_b0, mass 0.01; collision sphere radius=0.05; visual sphere radius=0.05
- added link eye_b1, mass 0.01; collision sphere radius=0.05; visual sphere radius=0.05
- added link leg_0_body0, mass 0.05; collision box size=0.1 0.2 0.1; visual box size=0.1 0.2 0.1
- added link leg_0_body1, mass 0.05; collision box size=0.1 0.2 0.1; visual box size=0.1 0.2 0.1
- added link leg_0_body2, mass 0.05; collision box size=0.1 0.2 0.1; visual box size=0.1 0.2 0.1
- added link leg_0_body3, mass 0.05; collision box size=0.1 0.2 0.1; visual box size=0.1 0.2 0.1
- added link leg_1_body0, mass 0.05; collision box size=0.1 0.2 0.1; visual box size=0.1 0.2 0.1
- added link leg_1_body1, mass 0.05; collision box size=0.1 0.2 0.1; visual box size=0.1 0.2 0.1
- added link leg_1_body2, mass 0.05; collision box size=0.1 0.2 0.1; visual box size=0.1 0.2 0.1
- added link leg_1_body3, mass 0.05; collision box size=0.1 0.2 0.1; visual box size=0.1 0.2 0.1
- added link leg_2_body0, mass 0.05; collision box size=0.1 0.2 0.1; visual box size=0.1 0.2 0.1
- added link leg_2_body1, mass 0.05; collision box size=0.1 0.2 0.1; visual box size=0.1 0.2 0.1
- added link leg_2_body2, mass 0.05; collision box size=0.1 0.2 0.1; visual box size=0.1 0.2 0.1
- added link leg_2_body3, mass 0.05; collision box size=0.1 0.2 0.1; visual box size=0.1 0.2 0.1
- added link leg_3_body0, mass 0.05; collision box size=0.1 0.2 0.1; visual box size=0.1 0.2 0.1
- added link leg_3_body1, mass 0.05; collision box size=0.1 0.2 0.1; visual box size=0.1 0.2 0.1
- added link leg_3_body2, mass 0.05; collision box size=0.1 0.2 0.1; visual box size=0.1 0.2 0.1
- added link leg_3_body3, mass 0.05; collision box size=0.1 0.2 0.1; visual box size=0.1 0.2 0.1
- added link leg_4_body0, mass 0.05; collision box size=0.1 0.2 0.1; visual box size=0.1 0.2 0.1
- added link leg_4_body1, mass 0.05; collision box size=0.1 0.2 0.1; visual box size=0.1 0.2 0.1
- added link leg_4_body2, mass 0.05; collision box size=0.1 0.2 0.1; visual box size=0.1 0.2 0.1
- added link leg_4_body3, mass 0.05; collision box size=0.1 0.2 0.1; visual box size=0.1 0.2 0.1
- added link leg_5_body0, mass 0.05; collision box size=0.1 0.2 0.1; visual box size=0.1 0.2 0.1
- added link leg_5_body1, mass 0.05; collision box size=0.1 0.2 0.1; visual box size=0.1 0.2 0.1
- added link leg_5_body2, mass 0.05; collision box size=0.1 0.2 0.1; visual box size=0.1 0.2 0.1
- added link leg_5_body3, mass 0.05; collision box size=0.1 0.2 0.1; visual box size=0.1 0.2 0.1
Joints:
- removed joint left_eye_joint
- removed joint leg0_joint0
- removed joint leg0_joint1
- removed joint leg0_joint2
- removed joint leg0_joint3
- removed joint leg1_joint0
- removed joint leg1_joint1
- removed joint leg1_joint2
- removed joint leg1_joint3
- removed joint leg2_joint0
- removed joint leg2_joint1
- removed joint leg2_joint2
- removed joint leg2_joint3
- removed joint leg3_joint0
- removed joint leg3_joint1
- removed joint leg3_joint2
- removed joint leg3_joint3
- removed joint leg4_joint0
- removed joint leg4_joint1
- removed joint leg4_joint2
- removed joint leg4_joint3
- removed joint leg5_joint0
- removed joint leg5_joint1
- removed joint leg5_joint2
- removed joint leg5_joint3
- removed joint neck_joint
- removed joint right_eye_joint
- added joint eye_j0: type fixed, parent head, child eye_b0, origin xyz=0.1 0.1 0.05 rpy=0 0 0
- added joint eye_j1: type fixed, parent head, child eye_b1, origin xyz=0.1 -0.1 0.05 rpy=0 0 0
- added joint leg_0_joint0: type fixed, parent body, child leg_0_body0, origin xyz=0.45 0.2 -0.1 rpy=0 0 0
- added joint leg_0_joint1: type revolute, parent leg_0_body0, child leg_0_body1, origin xyz=0 0.12 0 rpy=0 0 0, axis 0 1 0, limit lower=-0.79 upper=0.79 effort=10 velocity=1
- added joint leg_0_joint2: type revolute, parent leg_0_body1, child leg_0_body2, origin xyz=0 0.12 0 rpy=0 0 0, axis 1 0 0, limit lower=0 upper=1.05 effort=10 velocity=1
- added joint leg_0_joint3: type revolute, parent leg_0_body2, child leg_0_body3, origin xyz=0 0.12 0 rpy=0 0 0, axis 1 0 0, limit lower=0 upper=1.05 effort=10 velocity=1
- added joint leg_1_joint0: type fixed, parent body, child leg_1_body0, origin xyz=0 0.2 -0.1 rpy=0 0 0
- added joint leg_1_joint1: type revolute, parent leg_1_body0, child leg_1_body1, origin xyz=0 0.12 0 rpy=0 0 0, axis 0 1 0, limit lower=-0.79 upper=0.79 effort=10 velocity=1
- added joint leg_1_joint2: type revolute, parent leg_1_body1, child leg_1_body2, origin xyz=0 0.12 0 rpy=0 0 0, axis 1 0 0, limit lower=0 upper=1.05 effort=10 velocity=1
- added joint leg_1_joint3: type revolute, parent leg_1_body2, child leg_1_body3, origin xyz=0 0.12 0 rpy=0 0 0, axis 1 0 0, limit lower=0 upper=1.05 effort=10 velocity=1
- added joint leg_2_joint0: type fixed, parent body, child leg_2_body0, origin xyz=-0.45 0.2 -0.1 rpy=0 0 0
- added joint leg_2_joint1: type revolute, parent leg_2_body0, child leg_2_body1, origin xyz=0 0.12 0 rpy=0 0 0, axis 0 1 0, limit lower=-0.79 upper=0.79 effort=10 velocity=1
- added joint leg_2_joint2: type revolute, parent leg_2_body1, child leg_2_body2, origin xyz=0 0.12 0 rpy=0 0 0, axis 1 0 0, limit lower=0 upper=1.05 effort=10 velocity=1
- added joint leg_2_joint3: type revolute, parent leg_2_body2, child leg_2_body3, origin xyz=0 0.12 0 rpy=0 0 0, axis 1 0 0, limit lower=0 upper=1.05 effort=10 velocity=1
- added joint leg_3_joint0: type fixed, parent body, child leg_3_body0, origin xyz=0.45 -0.2 -0.1 rpy=0 0 3.14159
- added joint leg_3_joint1: type revolute, parent leg_3_body0, child leg_3_body1, origin xyz=0 0.12 0 rpy=0 0 0, axis 0 1 0, limit lower=-0.79 upper=0.79 effort=10 velocity=1
- added joint leg_3_joint2: type revolute, parent leg_3_body1, child leg_3_body2, origin xyz=0 0.12 0 rpy=0 0 0, axis 1 0 0, limit lower=0 upper=1.05 effort=10 velocity=1
- added joint leg_3_joint3: type revolute, parent leg_3_body2, child leg_3_body3, origin xyz=0 0.12 0 rpy=0 0 0, axis 1 0 0, limit lower=0 upper=1.05 effort=10 velocity=1
- added joint leg_4_joint0: type fixed, parent body, child leg_4_body0, origin xyz=0 -0.2 -0.1 rpy=0 0 3.14159
- added joint leg_4_joint1: type revolute, parent leg_4_body0, child leg_4_body1, origin xyz=0 0.12 0 rpy=0 0 0, axis 0 1 0, limit lower=-0.79 upper=0.79 effort=10 velocity=1
- added joint leg_4_joint2: type revolute, parent leg_4_body1, child leg_4_body2, origin xyz=0 0.12 0 rpy=0 0 0, axis 1 0 0, limit lower=0 upper=1.05 effort=10 velocity=1
- added joint leg_4_joint3: type revolute, parent leg_4_body2, child leg_4_body3, origin xyz=0 0.12 0 rpy=0 0 0, axis 1 0 0, limit lower=0 upper=1.05 effort=10 velocity=1
- added joint leg_5_joint0: type fixed, parent body, child leg_5_body0, origin xyz=-0.45 -0.2 -0.1 rpy=0 0 3.14159
- added joint leg_5_joint1: type revolute, parent leg_5_body0, child leg_5_body1, origin xyz=0 0.12 0 rpy=0 0 0, axis 0 1 0, limit lower=-0.79 upper=0.79 effort=10 velocity=1
- added joint leg_5_joint2: type revolute, parent leg_5_body1, child leg_5_body2, origin xyz=0 0.12 0 rpy=0 0 0, axis 1 0 0, limit lower=0 upper=1.05 effort=10 velocity=1
- added joint leg_5_joint3: type revolute, parent leg_5_body2, child leg_5_body3, origin xyz=0 0.12 0 rpy=0 0 0, axis 1 0 0, limit lower=0 upper=1.05 effort=10 velocity=1
- added joint neck_j: type fixed, parent body, child head, origin xyz=0.5 0 0.15 rpy=0 0 0

Commit message: feat: Standardize leg naming and joint definitions in hexapod URDF

File: models/hexapod.urdf (robot description, URDF)
Before this commit: robot hexapod, 28 links, 27 joints
Links:
- removed link leg_0_body0
- removed link leg_0_body1
- removed link leg_0_body2
- removed link leg_0_body3
- removed link leg_1_body0
- removed link leg_1_body1
- removed link leg_1_body2
- removed link leg_1_body3
- removed link leg_2_body0
- removed link leg_2_body1
- removed link leg_2_body2
- removed link leg_2_body3
- removed link leg_3_body0
- removed link leg_3_body1
- removed link leg_3_body2
- removed link leg_3_body3
- removed link leg_4_body0
- removed link leg_4_body1
- removed link leg_4_body2
- removed link leg_4_body3
- removed link leg_5_body0
- removed link leg_5_body1
- removed link leg_5_body2
- removed link leg_5_body3
- added link leg0_body0, mass 0.05; collision box size=0.1 0.2 0.1; visual box size=0.1 0.2 0.1
- added link leg0_body1, mass 0.05; collision box size=0.1 0.2 0.1; visual box size=0.1 0.2 0.1
- added link leg0_body2, mass 0.05; collision box size=0.1 0.2 0.1; visual box size=0.1 0.2 0.1
- added link leg1_body0, mass 0.05; collision box size=0.1 0.2 0.1; visual box size=0.1 0.2 0.1
- added link leg1_body1, mass 0.05; collision box size=0.1 0.2 0.1; visual box size=0.1 0.2 0.1
- added link leg1_body2, mass 0.05; collision box size=0.1 0.2 0.1; visual box size=0.1 0.2 0.1
- added link leg2_body0, mass 0.05; collision box size=0.1 0.2 0.1; visual box size=0.1 0.2 0.1
- added link leg2_body1, mass 0.05; collision box size=0.1 0.2 0.1; visual box size=0.1 0.2 0.1
- added link leg2_body2, mass 0.05; collision box size=0.1 0.2 0.1; visual box size=0.1 0.2 0.1
- added link leg3_body0, mass 0.05; collision box size=0.1 0.2 0.1; visual box size=0.1 0.2 0.1
- added link leg3_body1, mass 0.05; collision box size=0.1 0.2 0.1; visual box size=0.1 0.2 0.1
- added link leg3_body2, mass 0.05; collision box size=0.1 0.2 0.1; visual box size=0.1 0.2 0.1
- added link leg4_body0, mass 0.05; collision box size=0.1 0.2 0.1; visual box size=0.1 0.2 0.1
- added link leg4_body1, mass 0.05; collision box size=0.1 0.2 0.1; visual box size=0.1 0.2 0.1
- added link leg4_body2, mass 0.05; collision box size=0.1 0.2 0.1; visual box size=0.1 0.2 0.1
- added link leg5_body0, mass 0.05; collision box size=0.1 0.2 0.1; visual box size=0.1 0.2 0.1
- added link leg5_body1, mass 0.05; collision box size=0.1 0.2 0.1; visual box size=0.1 0.2 0.1
- added link leg5_body2, mass 0.05; collision box size=0.1 0.2 0.1; visual box size=0.1 0.2 0.1
Joints:
- removed joint leg_0_joint0
- removed joint leg_0_joint1
- removed joint leg_0_joint2
- removed joint leg_0_joint3
- removed joint leg_1_joint0
- removed joint leg_1_joint1
- removed joint leg_1_joint2
- removed joint leg_1_joint3
- removed joint leg_2_joint0
- removed joint leg_2_joint1
- removed joint leg_2_joint2
- removed joint leg_2_joint3
- removed joint leg_3_joint0
- removed joint leg_3_joint1
- removed joint leg_3_joint2
- removed joint leg_3_joint3
- removed joint leg_4_joint0
- removed joint leg_4_joint1
- removed joint leg_4_joint2
- removed joint leg_4_joint3
- removed joint leg_5_joint0
- removed joint leg_5_joint1
- removed joint leg_5_joint2
- removed joint leg_5_joint3
- added joint knee_back_leftL_link: type revolute, parent leg2_body1, child leg2_body2, origin xyz=0 0.12 0 rpy=0 0 0, axis 1 0 0, limit lower=0 upper=1.05 effort=10 velocity=1
- added joint knee_back_rightR_link: type revolute, parent leg5_body1, child leg5_body2, origin xyz=0 0.12 0 rpy=0 0 0, axis 1 0 0, limit lower=0 upper=1.05 effort=10 velocity=1
- added joint knee_front_leftL_link: type revolute, parent leg0_body1, child leg0_body2, origin xyz=0 0.12 0 rpy=0 0 0, axis 1 0 0, limit lower=0 upper=1.05 effort=10 velocity=1
- added joint knee_front_leftR_link: type revolute, parent leg1_body1, child leg1_body2, origin xyz=0 0.12 0 rpy=0 0 0, axis 1 0 0, limit lower=0 upper=1.05 effort=10 velocity=1
- added joint knee_front_rightL_link: type revolute, parent leg3_body1, child leg3_body2, origin xyz=0 0.12 0 rpy=0 0 0, axis 1 0 0, limit lower=0 upper=1.05 effort=10 velocity=1
- added joint knee_front_rightR_link: type revolute, parent leg4_body1, child leg4_body2, origin xyz=0 0.12 0 rpy=0 0 0, axis 1 0 0, limit lower=0 upper=1.05 effort=10 velocity=1
- added joint motor_back_leftL_joint: type fixed, parent body, child leg2_body0, origin xyz=-0.45 0.2 0 rpy=0 0 0
- added joint motor_back_leftR_joint: type revolute, parent leg2_body0, child leg2_body1, origin xyz=0 0.12 0 rpy=0 0 0, axis 0 1 0, limit lower=-0.79 upper=0.79 effort=10 velocity=1
- added joint motor_back_rightL_joint: type fixed, parent body, child leg5_body0, origin xyz=-0.45 -0.2 0 rpy=0 0 3.14159
- added joint motor_back_rightL_joint2: type fixed, parent body, child leg4_body0, origin xyz=0 -0.2 0 rpy=0 0 3.14159
- added joint motor_back_rightR_joint: type revolute, parent leg5_body0, child leg5_body1, origin xyz=0 0.12 0 rpy=0 0 0, axis 0 1 0, limit lower=-0.79 upper=0.79 effort=10 velocity=1
- added joint motor_back_rightR_joint2: type revolute, parent leg4_body0, child leg4_body1, origin xyz=0 0.12 0 rpy=0 0 0, axis 0 1 0, limit lower=-0.79 upper=0.79 effort=10 velocity=1
- added joint motor_front_leftL_joint: type fixed, parent body, child leg0_body0, origin xyz=0.45 0.2 0 rpy=0 0 0
- added joint motor_front_leftL_joint2: type fixed, parent body, child leg1_body0, origin xyz=0 0.2 0 rpy=0 0 0
- added joint motor_front_leftR_joint: type revolute, parent leg0_body0, child leg0_body1, origin xyz=0 0.12 0 rpy=0 0 0, axis 0 1 0, limit lower=-0.79 upper=0.79 effort=10 velocity=1
- added joint motor_front_leftR_joint2: type revolute, parent leg1_body0, child leg1_body1, origin xyz=0 0.12 0 rpy=0 0 0, axis 0 1 0, limit lower=-0.79 upper=0.79 effort=10 velocity=1
- added joint motor_front_rightL_joint: type fixed, parent body, child leg3_body0, origin xyz=0.45 -0.2 0 rpy=0 0 3.14159
- added joint motor_front_rightR_joint: type revolute, parent leg3_body0, child leg3_body1, origin xyz=0 0.12 0 rpy=0 0 0, axis 0 1 0, limit lower=-0.79 upper=0.79 effort=10 velocity=1

Commit message: feat: Standardize joint naming in hexapod URDF and update robot control mappings

File: models/hexapod.urdf (robot description, URDF)
Before this commit: robot hexapod, 22 links, 21 joints
Joints:
- removed joint knee_back_leftL_link
- removed joint knee_back_rightR_link
- removed joint knee_front_leftL_link
- removed joint knee_front_leftR_link
- removed joint knee_front_rightL_link
- removed joint knee_front_rightR_link
- removed joint motor_back_leftL_joint
- removed joint motor_back_leftR_joint
- removed joint motor_back_rightL_joint
- removed joint motor_back_rightL_joint2
- removed joint motor_back_rightR_joint
- removed joint motor_back_rightR_joint2
- removed joint motor_front_leftL_joint
- removed joint motor_front_leftL_joint2
- removed joint motor_front_leftR_joint
- removed joint motor_front_leftR_joint2
- removed joint motor_front_rightL_joint
- removed joint motor_front_rightR_joint
- added joint knee_back_left_joint: type revolute, parent leg2_body1, child leg2_body2, origin xyz=0 0.12 0 rpy=0 0 0, axis 1 0 0, limit lower=0 upper=1.05 effort=10 velocity=1
- added joint knee_back_right_joint: type revolute, parent leg5_body1, child leg5_body2, origin xyz=0 0.12 0 rpy=0 0 0, axis 1 0 0, limit lower=0 upper=1.05 effort=10 velocity=1
- added joint knee_front_left_joint: type revolute, parent leg0_body1, child leg0_body2, origin xyz=0 0.12 0 rpy=0 0 0, axis 1 0 0, limit lower=0 upper=1.05 effort=10 velocity=1
- added joint knee_front_right_joint: type revolute, parent leg3_body1, child leg3_body2, origin xyz=0 0.12 0 rpy=0 0 0, axis 1 0 0, limit lower=0 upper=1.05 effort=10 velocity=1
- added joint knee_middle_left_joint: type revolute, parent leg1_body1, child leg1_body2, origin xyz=0 0.12 0 rpy=0 0 0, axis 1 0 0, limit lower=0 upper=1.05 effort=10 velocity=1
- added joint knee_middle_right_joint: type revolute, parent leg4_body1, child leg4_body2, origin xyz=0 0.12 0 rpy=0 0 0, axis 1 0 0, limit lower=0 upper=1.05 effort=10 velocity=1
- added joint motor_back_left_base_joint: type fixed, parent body, child leg2_body0, origin xyz=-0.45 0.2 0 rpy=0 0 0
- added joint motor_back_left_joint: type revolute, parent leg2_body0, child leg2_body1, origin xyz=0 0.12 0 rpy=0 0 0, axis 0 1 0, limit lower=-0.79 upper=0.79 effort=10 velocity=1
- added joint motor_back_right_base_joint: type fixed, parent body, child leg5_body0, origin xyz=-0.45 -0.2 0 rpy=0 0 3.14159
- added joint motor_back_right_joint: type revolute, parent leg5_body0, child leg5_body1, origin xyz=0 0.12 0 rpy=0 0 0, axis 0 1 0, limit lower=-0.79 upper=0.79 effort=10 velocity=1
- added joint motor_front_left_base_joint: type fixed, parent body, child leg0_body0, origin xyz=0.45 0.2 0 rpy=0 0 0
- added joint motor_front_left_joint: type revolute, parent leg0_body0, child leg0_body1, origin xyz=0 0.12 0 rpy=0 0 0, axis 0 1 0, limit lower=-0.79 upper=0.79 effort=10 velocity=1
- added joint motor_front_right_base_joint: type fixed, parent body, child leg3_body0, origin xyz=0.45 -0.2 0 rpy=0 0 3.14159
- added joint motor_front_right_joint: type revolute, parent leg3_body0, child leg3_body1, origin xyz=0 0.12 0 rpy=0 0 0, axis 0 1 0, limit lower=-0.79 upper=0.79 effort=10 velocity=1
- added joint motor_middle_left_base_joint: type fixed, parent body, child leg1_body0, origin xyz=0 0.2 0 rpy=0 0 0
- added joint motor_middle_left_joint: type revolute, parent leg1_body0, child leg1_body1, origin xyz=0 0.12 0 rpy=0 0 0, axis 0 1 0, limit lower=-0.79 upper=0.79 effort=10 velocity=1
- added joint motor_middle_right_base_joint: type fixed, parent body, child leg4_body0, origin xyz=0 -0.2 0 rpy=0 0 3.14159
- added joint motor_middle_right_joint: type revolute, parent leg4_body0, child leg4_body1, origin xyz=0 0.12 0 rpy=0 0 0, axis 0 1 0, limit lower=-0.79 upper=0.79 effort=10 velocity=1
