Commit message: feat: Refactor hexapod URDF to standardize joint naming and improve material definitions

File: models/hexapod.urdf (robot description, URDF)
Before this commit: robot hexapod, 22 links, 21 joints
Links:
- removed link body
- removed link eye_b0
- removed link eye_b1
- removed link leg0_body0
- removed link leg0_body1
- removed link leg0_body2
- removed link leg1_body0
- removed link leg1_body1
- removed link leg1_body2
- removed link leg2_body0
- removed link leg2_body1
- removed link leg2_body2
- removed link leg3_body0
- removed link leg3_body1
- removed link leg3_body2
- removed link leg4_body0
- removed link leg4_body1
- removed link leg4_body2
- removed link leg5_body0
- removed link leg5_body1
- removed link leg5_body2
- added link base_link, mass 1.0; collision box size=1.0 0.4 0.2; visual box size=1.0 0.4 0.2
- added link elbow_back_left, mass 0.05; collision box size=0.1 0.2 0.1; visual box size=0.1 0.2 0.1
- added link elbow_back_right, mass 0.05; collision box size=0.1 0.2 0.1; visual box size=0.1 0.2 0.1
- added link elbow_front_left, mass 0.05; collision box size=0.1 0.2 0.1; visual box size=0.1 0.2 0.1
- added link elbow_front_right, mass 0.05; collision box size=0.1 0.2 0.1; visual box size=0.1 0.2 0.1
- added link elbow_middle_left, mass 0.05; collision box size=0.1 0.2 0.1; visual box size=0.1 0.2 0.1
- added link elbow_middle_right, mass 0.05; collision box size=0.1 0.2 0.1; visual box size=0.1 0.2 0.1
- added link eye_left, mass 0.01; collision sphere radius=0.05; visual sphere radius=0.05
- added link eye_right, mass 0.01; collision sphere radius=0.05; visual sphere radius=0.05
- added link knee_back_left, mass 0.05; collision box size=0.1 0.2 0.1; visual box size=0.1 0.2 0.1
- added link knee_back_right, mass 0.05; collision box size=0.1 0.2 0.1; visual box size=0.1 0.2 0.1
- added link knee_front_left, mass 0.05; collision box size=0.1 0.2 0.1; visual box size=0.1 0.2 0.1
- added link knee_front_right, mass 0.05; collision box size=0.1 0.2 0.1; visual box size=0.1 0.2 0.1
- added link knee_middle_left, mass 0.05; collision box size=0.1 0.2 0.1; visual box size=0.1 0.2 0.1
- added link knee_middle_right, mass 0.05; collision box size=0.1 0.2 0.1; visual box size=0.1 0.2 0.1
- added link shoulder_back_left, mass 0.05; collision box size=0.1 0.2 0.1; visual box size=0.1 0.2 0.1
- added link shoulder_back_right, mass 0.05; collision box size=0.1 0.2 0.1; visual box size=0.1 0.2 0.1
- added link shoulder_front_left, mass 0.05; collision box size=0.1 0.2 0.1; visual box size=0.1 0.2 0.1
- added link shoulder_front_right, mass 0.05; collision box size=0.1 0.2 0.1; visual box size=0.1 0.2 0.1
- added link shoulder_middle_left, mass 0.05; collision box size=0.1 0.2 0.1; visual box size=0.1 0.2 0.1
- added link shoulder_middle_right, mass 0.05; collision box size=0.1 0.2 0.1; visual box size=0.1 0.2 0.1
Joints:
- removed joint eye_j0
- removed joint eye_j1
- removed joint motor_back_left_base_joint
- removed joint motor_back_left_joint
- removed joint motor_back_right_base_joint
- removed joint motor_back_right_joint
- removed joint motor_front_left_base_joint
- removed joint motor_front_left_joint
- removed joint motor_front_right_base_joint
- removed joint motor_front_right_joint
- removed joint motor_middle_left_base_joint
- removed joint motor_middle_left_joint
- removed joint motor_middle_right_base_joint
- removed joint motor_middle_right_joint
- removed joint neck_j
- added joint elbow_back_left_joint: type revolute, parent shoulder_back_left, child elbow_back_left, origin xyz=0 0.24 0 rpy=0 0 0, axis 1 0 0, limit lower=0 upper=1.047 effort=10 velocity=3
- added joint elbow_back_right_joint: type revolute, parent shoulder_back_right, child elbow_back_right, origin xyz=0 0.24 0 rpy=0 0 0, axis 1 0 0, limit lower=0 upper=1.047 effort=10 velocity=3
- added joint elbow_front_left_joint: type revolute, parent shoulder_front_left, child elbow_front_left, origin xyz=0 0.24 0 rpy=0 0 0, axis 1 0 0, limit lower=0 upper=1.047 effort=10 velocity=3
- added joint elbow_front_right_joint: type revolute, parent shoulder_front_right, child elbow_front_right, origin xyz=0 0.24 0 rpy=0 0 0, axis 1 0 0, limit lower=0 upper=1.047 effort=10 velocity=3
- added joint elbow_middle_left_joint: type revolute, parent shoulder_middle_left, child elbow_middle_left, origin xyz=0 0.24 0 rpy=0 0 0, axis 1 0 0, limit lower=0 upper=1.047 effort=10 velocity=3
- added joint elbow_middle_right_joint: type revolute, parent shoulder_middle_right, child elbow_middle_right, origin xyz=0 0.24 0 rpy=0 0 0, axis 1 0 0, limit lower=0 upper=1.047 effort=10 velocity=3
- added joint eye_left_joint: type fixed, parent head, child eye_left, origin xyz=0.1 0.1 0.05 rpy=0 0 0
- added joint eye_right_joint: type fixed, parent head, child eye_right, origin xyz=0.1 -0.1 0.05 rpy=0 0 0
- added joint head_joint: type fixed, parent base_link, child head, origin xyz=0.5 0 0.15 rpy=0 0 0
- added joint shoulder_back_left_joint: type revolute, parent base_link, child shoulder_back_left, origin xyz=-0.45 0.2 0.1 rpy=0 0 0, axis 0 1 0, limit lower=-0.785 upper=0.785 effort=10 velocity=3
- added joint shoulder_back_right_joint: type revolute, parent base_link, child shoulder_back_right, origin xyz=-0.45 -0.2 0.1 rpy=0 0 3.14159, axis 0 1 0, limit lower=-0.785 upper=0.785 effort=10 velocity=3
- added joint shoulder_front_left_joint: type revolute, parent base_link, child shoulder_front_left, origin xyz=0.45 0.2 0.1 rpy=0 0 0, axis 0 1 0, limit lower=-0.785 upper=0.785 effort=10 velocity=3
- added joint shoulder_front_right_joint: type revolute, parent base_link, child shoulder_front_right, origin xyz=0.45 -0.2 0.1 rpy=0 0 3.14159, axis 0 1 0, limit lower=-0.785 upper=0.785 effort=10 velocity=3
- added joint shoulder_middle_left_joint: type revolute, parent base_link, child shoulder_middle_left, origin xyz=0.0 0.2 0.1 rpy=0 0 0, axis 0 1 0, limit lower=-0.785 upper=0.785 effort=10 velocity=3
- added joint shoulder_middle_right_joint: type revolute, parent base_link, child shoulder_middle_right, origin xyz=0.0 -0.2 0.1 rpy=0 0 3.14159, axis 0 1 0, limit lower=-0.785 upper=0.785 effort=10 velocity=3
- joint knee_back_left_joint: child leg2_body2 -> knee_back_left; limit lower=0 upper=1.05 effort=10 velocity=1 -> lower=0 upper=1.047 effort=10 velocity=3; origin xyz=0 0.12 0 rpy=0 0 0 -> xyz=0 0.24 0 rpy=0 0 0; parent leg2_body1 -> elbow_back_left
- joint knee_back_right_joint: child leg5_body2 -> knee_back_right; limit lower=0 upper=1.05 effort=10 velocity=1 -> lower=0 upper=1.047 effort=10 velocity=3; origin xyz=0 0.12 0 rpy=0 0 0 -> xyz=0 0.24 0 rpy=0 0 0; parent leg5_body1 -> elbow_back_right
- joint knee_front_left_joint: child leg0_body2 -> knee_front_left; limit lower=0 upper=1.05 effort=10 velocity=1 -> lower=0 upper=1.047 effort=10 velocity=3; origin xyz=0 0.12 0 rpy=0 0 0 -> xyz=0 0.24 0 rpy=0 0 0; parent leg0_body1 -> elbow_front_left
- joint knee_front_right_joint: child leg3_body2 -> knee_front_right; limit lower=0 upper=1.05 effort=10 velocity=1 -> lower=0 upper=1.047 effort=10 velocity=3; origin xyz=0 0.12 0 rpy=0 0 0 -> xyz=0 0.24 0 rpy=0 0 0; parent leg3_body1 -> elbow_front_right
- joint knee_middle_left_joint: child leg1_body2 -> knee_middle_left; limit lower=0 upper=1.05 effort=10 velocity=1 -> lower=0 upper=1.047 effort=10 velocity=3; origin xyz=0 0.12 0 rpy=0 0 0 -> xyz=0 0.24 0 rpy=0 0 0; parent leg1_body1 -> elbow_middle_left
- joint knee_middle_right_joint: child leg4_body2 -> knee_middle_right; limit lower=0 upper=1.05 effort=10 velocity=1 -> lower=0 upper=1.047 effort=10 velocity=3; origin xyz=0 0.12 0 rpy=0 0 0 -> xyz=0 0.24 0 rpy=0 0 0; parent leg4_body1 -> elbow_middle_right

Commit message: feat: Update joint origin positions in hexapod URDF for consistency

File: models/hexapod.urdf (robot description, URDF)
Before this commit: robot hexapod, 22 links, 21 joints
Joints:
- joint shoulder_back_left_joint: origin xyz=-0.45 0.2 0.1 rpy=0 0 0 -> xyz=-0.45 0.2 0 rpy=0 0 0
- joint shoulder_back_right_joint: origin xyz=-0.45 -0.2 0.1 rpy=0 0 3.14159 -> xyz=-0.45 -0.2 0 rpy=0 0 3.14159
- joint shoulder_front_left_joint: origin xyz=0.45 0.2 0.1 rpy=0 0 0 -> xyz=0.45 0.2 0 rpy=0 0 0
- joint shoulder_front_right_joint: origin xyz=0.45 -0.2 0.1 rpy=0 0 3.14159 -> xyz=0.45 -0.2 0 rpy=0 0 3.14159
- joint shoulder_middle_left_joint: origin xyz=0.0 0.2 0.1 rpy=0 0 0 -> xyz=0.0 0.2 0 rpy=0 0 0
- joint shoulder_middle_right_joint: origin xyz=0.0 -0.2 0.1 rpy=0 0 3.14159 -> xyz=0.0 -0.2 0 rpy=0 0 3.14159

Commit message: feat: Reverse joint axis direction for front and middle left legs in hexapod URDF

File: models/hexapod.urdf (robot description, URDF)
Before this commit: robot hexapod, 22 links, 21 joints
Joints:
- joint elbow_back_left_joint: axis 1 0 0 -> -1 0 0
- joint elbow_back_right_joint: axis 1 0 0 -> -1 0 0
- joint elbow_front_left_joint: axis 1 0 0 -> -1 0 0
- joint elbow_front_right_joint: axis 1 0 0 -> -1 0 0
- joint elbow_middle_left_joint: axis 1 0 0 -> -1 0 0
- joint elbow_middle_right_joint: axis 1 0 0 -> -1 0 0
- joint knee_back_left_joint: axis 1 0 0 -> -1 0 0
- joint knee_back_right_joint: axis 1 0 0 -> -1 0 0
- joint knee_front_left_joint: axis 1 0 0 -> -1 0 0
- joint knee_front_right_joint: axis 1 0 0 -> -1 0 0
- joint knee_middle_left_joint: axis 1 0 0 -> -1 0 0
- joint knee_middle_right_joint: axis 1 0 0 -> -1 0 0
